File: electrical/pcb/control_board/Control_Boards.kicad_pcb (KiCad board)
At the start: 2 copper layers, 220 x 329.2 mm, 148 parts, among them J1 XT30-M, J10 Molex_172675-0613, J11 Molex_172675-0613, J12 TSW-104-07-F-T, J13 Molex_172675-0613, J14 Molex_172675-0613, J16 277-11404-ND, J17 277-11404-ND, J18 277-11404-ND, J19 TSW-104-07-F-T, J2 ED2580-ND, J20 PEC08SAAN, J21 PPTC102LFBN-RC, J22 S9175-ND_rpi_breakout, J23 S9175-ND_rpi_breakout, J24 6posheader, J25 SSW-104-01-F-T, J26 WM6548-ND, J27 PPTC021LFBN-RC, J28 PPTC021LFBN-RC, J29 PPTC021LFBN-RC, J3 XT30-F, J30 PEC08SAAN, J4 XT30-F, J5 XT30-M, J6 ED2580-ND, J7 TSW-104-07-F-T, J8 Molex_172675-0613, J9 Molex_172675-0613, M1 Mounting_Holes, Q1 2N3906, Q2 2N3906, Q3 2N3906, Q4 2N3906, Q5 2N3906, Q6 2N3906, SW1 CT206124-ND, T1 test_point, T10 test_point, T11 test_point, T12 test_point, T13 test_point, T14 test_point, T15 test_point, T2 test_point, T3 test_point, T4 test_point, T5 test_point, T6 test_point, T7 test_point, T8 test_point, T9 test_point, U1 INA260, U2 PCA9685, U3 D24V22Fx, U4 D24V150Fx, U5 DC7G3HWA, U6 DC7G3HWA, U7 MIC2937A-3.3WT, y1 rover_silkscreen, y2 rover_silkscreen

Commit message: update to kicad10, bump rev on back of motor board to v2.0.3
Other:
- board text added: "Open Source Rover Robotic Breakout Boards Brain Board v2.0.3"
- board text removed: "Open Source Rover Robotic Breakout Boards Brain Board v2.0.2"

Commit message: updated export_schematic script to expand ${VERSION} properly, plus new schematics and 3d_images
Other:
- board text added: "Open Source Rover Robotic Breakout Boards - Brain Board - ${VERSION}"
- board text added: "Open Source Rover Robotic Breakout Boards Brain Board ${VERSION}"
- board text added: "Open Source Rover Robotic Breakout Boards Motor Board - ${VERSION}"
- board text removed: "Open Source Rover Robotic Breakout Boards - Brain Board - v2.0.3"
- board text removed: "Open Source Rover Robotic Breakout Boards Brain Board v2.0.3"
- board text removed: "Open Source Rover Robotic Breakout Boards Motor Board - v2.0.3"
Changed lines of the file:
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@@
 		)
 	)
-	(gr_text "Open Source Rover\nRobotic Breakout Boards\nMotor Board - v2.0.3"
+	(gr_text "Open Source Rover\nRobotic Breakout Boards\nMotor Board - ${VERSION}"
 		(at 109.892349 -17.5006 0)
 		(layer "F.SilkS")
@@
 		)
 	)
-	(gr_text "Open Source Rover \nRobotic Breakout Boards - Brain Board - v2.0.3"
+	(gr_text "Open Source Rover \nRobotic Breakout Boards - Brain Board - ${VERSION}"
 		(at 126.2126 -226.822 0)
 		(layer "F.SilkS")
@@
 		)
 	)
-	(gr_text "Open Source Rover\nRobotic Breakout Boards\nBrain Board\nv2.0.3"
+	(gr_text "Open Source Rover\nRobotic Breakout Boards\nBrain Board\n${VERSION}"
 		(at 125.0442 -196.2404 0)
 		(layer "B.SilkS")
